Commit message: remove LMS1xx

File: ridgeback_description/urdf/accessories.urdf.xacro (robot description, xacro)
@@ -9,6 +9,4 @@
     ridgeback_base/launch/base.launch
   -->
-  <xacro:include filename="$(find ridgeback_description)/urdf/accessories/sick_lms1xx_mount.urdf.xacro" />
-  <xacro:include filename="$(find ridgeback_description)/urdf/accessories/sick_s300_mount.urdf.xacro" />
   <xacro:include filename="$(find ridgeback_description)/urdf/accessories/hokuyo_ust-10lx_mount.urdf.xacro" />
   <!-- If enabled, generate the front HOKUYO UST-10LX LASER payload. -->
@@ -24,38 +22,3 @@
                                  location="-1" />
   </xacro:if>
-  <!-- If enabled, generate the front SICK LMS111 LASER payload. -->
-  <xacro:if value="$(optenv RIDGEBACK_FRONT_SICK_LASER 0)">
-    <xacro:sick_lms1xx_mount prefix="/front"
-                             topic="/front/scan"
-                             location="1" />
-  </xacro:if>
-  <!-- If enabled, generate the rear SICK LMS111 LASER payload. -->
-  <xacro:if value="$(optenv RIDGEBACK_REAR_SICK_LASER 0)">
-    <xacro:sick_lms1xx_mount prefix="/rear"
-                             topic="/rear/scan"
-                             location="-1" />
-  </xacro:if>
-  <!-- If enabled, generate the front SICK S300 LASER payload.
-       This uses the same mesh as the lms1xx since they are the footprint
-       and the simulation parameters can be variable. -->
-  <xacro:if value="$(optenv RIDGEBACK_FRONT_S300_LASER 0)">
-    <xacro:sick_s300_mount prefix="/front"
-                             topic="/front/scan"
-                             location="1" />
-  </xacro:if>
-  <!-- If enabled, generate the rear SICK S300 LASER payload. -->
-  <xacro:if value="$(optenv RIDGEBACK_REAR_S300_LASER 0)">
-    <xacro:sick_s300_mount prefix="/rear"
-                             topic="/rear/scan"
-                             location="-1" />
-  </xacro:if>
-  <!-- If enabled, generate the optional Microstrain 3DM-GX2/3 IMU payload. -->
-  <xacro:include filename="$(find ridgeback_description)/urdf/accessories/microstrain_imu.urdf.xacro" />
-  <xacro:if value="$(optenv RIDGEBACK_MICROSTRAIN_IMU 0)">
-    <xacro:microstrain_imu prefix="$(optenv RIDGEBACK_MICROSTRAIN_IMU_PREFIX upgraded)"
-                           mount_link="$(optenv RIDGEBACK_MICROSTRAIN_IMU_MOUNT mid)_mount" >
-      <origin xyz="$(optenv RIDGEBACK_MICROSTRAIN_IMU_OFFSET 0 0 0)"
-              rpy="$(optenv RIDGEBACK_MICROSTRAIN_IMU_RPY 0 0 0)" />
-    </xacro:microstrain_imu>
-  </xacro:if>
 </robot>
